File: Distiller Controller V6/Pissbot/_autosave-Pissbot.sch (KiCad schematic (older format))
At the start: 62 parts, among them J1 Raspberry_Pi_2_3, J2 T1, J3 T5, J4 T2, J5 T6, J6 T3, J7 T7, J8 T4, J9 T8, U1 CP2102-GM, U2 TPS563231DRLR, U3 TLV74033PDBVR

Commit message: Updated PCB. Added library files
Parts:
- removed C?: 0.1uF, symbol Device:C_Small
- removed J?: MicroUSB_PI, symbol Connector:USB_B_Micro
- removed R8: 2k, symbol Device:R_Small
- removed U?: MCP23017_ML, Package_DFN_QFN:QFN-28-1EP_6x6mm_P0.65mm_EP4.25x4.25mm, symbol Interface_Expansion:MCP23017_ML
- added J11, J12, J13: T4, JST-SH 3 Connector:JST_SM03B-SRSS-TB(LF)(SN), symbol Pissbot-rescue:SM03B-SRSS-TB(LF)(SN)-SM03B-SRSS-TB_LF__SN_
- added J14, J15: SM02B-SRSS-TB(LF)(SN), JST SH 2Pin:SM02B-SRSS-TB(LF)(SN), symbol SM02B-SRSS-TB_LF__SN_:SM02B-SRSS-TB(LF)(SN)
- added J16: Conn_01x02_Female, Connector_AMASS:AMASS_XT30PW-F_1x02_P2.50mm_Horizontal, symbol Connector:Conn_01x02_Female
- added J17, J18: Conn_01x02_Female, Screw Terminal - TB001:CUI_TB001-500-02BE, symbol Connector:Conn_01x02_Female
- added R17, R18, R19, R20, R?: 2k, Resistor_SMD:R_0603_1608Metric_Pad1.05x0.95mm_HandSolder, symbol Pissbot-rescue:R_Small-Device
- added U? (x2): PTS647SM38SMTR2LFS, SW_PTS647SM38SMTR2LFS_CNK, symbol TactileSwitch:PTS647SM38SMTR2LFS
- A1: footprint XCVR_ESP32-WROVER-I -> ESP32-WROVER-I:XCVR_ESP32-WROVER-I; symbol ESP32-WROVER-I:ESP32-WROVER-I -> Pissbot-rescue:ESP32-WROVER-I-ESP32-WROVER-I
- C1: footprint (none) -> Capacitor_SMD:C_0603_1608Metric
- C10, C11, C5, C6, C9: footprint (none) -> Capacitor_SMD:C_0603_1608Metric; symbol Device:C_Small -> Pissbot-rescue:C_Small-Device
- C12, C13, C14: renamed from C?; footprint (none) -> Capacitor_SMD:C_0603_1608Metric; symbol Device:C_Small -> Pissbot-rescue:C_Small-Device
- C2: renamed from C3; footprint (none) -> Capacitor_SMD:C_0603_1608Metric; symbol Device:C_Small -> Pissbot-rescue:C_Small-Device
- C3: renamed from C4; footprint (none) -> Capacitor_SMD:C_0603_1608Metric; symbol Device:C_Small -> Pissbot-rescue:C_Small-Device
- C4: renamed from C2; footprint (none) -> Capacitor_SMD:C_0603_1608Metric
- C7: renamed from C8; footprint (none) -> Capacitor_SMD:C_0603_1608Metric; symbol Device:C_Small -> Pissbot-rescue:C_Small-Device
- C8: renamed from C7; footprint (none) -> Capacitor_SMD:C_0603_1608Metric
- D1: footprint (none) -> LED_SMD:LED_0201_0603Metric; symbol Device:LED_Small -> Pissbot-rescue:LED_Small-Device
- D2, D3: renamed from D?; footprint (none) -> Package_TO_SOT_SMD:TO-252-2; symbol Device:D_Schottky -> Pissbot-rescue:D_Schottky-Device
- D4, D5, D6: renamed from D?; footprint (none) -> Package_TO_SOT_SMD:SOT-23; symbol Device:D_Zener_Small_ALT -> Pissbot-rescue:D_Zener_Small_ALT-Device
- J1: renamed from J2; footprint JST_SM03B-SRSS-TB(LF)(SN) -> JST-SH 3 Connector:JST_SM03B-SRSS-TB(LF)(SN)
- J10: renamed from J1; footprint (none) -> PiZero:ADA3708_RPI-ZERO
- J2: renamed from J3; footprint JST_SM03B-SRSS-TB(LF)(SN) -> JST-SH 3 Connector:JST_SM03B-SRSS-TB(LF)(SN)
- J3: renamed from J4; footprint JST_SM03B-SRSS-TB(LF)(SN) -> JST-SH 3 Connector:JST_SM03B-SRSS-TB(LF)(SN)
- J4: renamed from J5; footprint JST_SM03B-SRSS-TB(LF)(SN) -> JST-SH 3 Connector:JST_SM03B-SRSS-TB(LF)(SN)
- J5: renamed from J6; footprint JST_SM03B-SRSS-TB(LF)(SN) -> JST-SH 3 Connector:JST_SM03B-SRSS-TB(LF)(SN)
- J6: renamed from J7; footprint JST_SM03B-SRSS-TB(LF)(SN) -> JST-SH 3 Connector:JST_SM03B-SRSS-TB(LF)(SN)
- J7: renamed from J8; footprint JST_SM03B-SRSS-TB(LF)(SN) -> JST-SH 3 Connector:JST_SM03B-SRSS-TB(LF)(SN)
- J8: renamed from J9; footprint JST_SM03B-SRSS-TB(LF)(SN) -> JST-SH 3 Connector:JST_SM03B-SRSS-TB(LF)(SN)
- J9: renamed from J?; footprint (none) -> Micro USB:Micro-USB-TE_2040002-1; symbol Connector:USB_B_Micro -> Pissbot-rescue:USB_B_Micro-Connector
- L1: footprint (none) -> 3_3uH_ECSMPIL06303R3MC:ECS-MPIL0630-3R3MC
- Q1, Q2: renamed from Q?; footprint (none) -> Package_TO_SOT_SMD:TO-252-2; symbol Device:Q_NMOS_GDS -> Pissbot-rescue:Q_NMOS_GDS-Device
- Q3, Q4, Q5: renamed from Q?; footprint SOT-23F_TOS -> Package_TO_SOT_SMD:SOT-23; symbol SSM3J338R:SSM3J338R -> Pissbot-rescue:SSM3J338R-SSM3J338R
- Q6, Q7: renamed from Q?; footprint Package_TO_SOT_THT:TO-92_Inline -> Package_TO_SOT_SMD:SOT-23; symbol Transistor_BJT:S8050 -> Pissbot-rescue:S8050-Transistor_BJT
- R1, R2, R3, R4: footprint (none) -> Resistor_SMD:R_0603_1608Metric_Pad1.05x0.95mm_HandSolder
- R10, R11, R12, R13, R14, R15, R16, R9: renamed from R?; footprint (none) -> Resistor_SMD:R_0603_1608Metric_Pad1.05x0.95mm_HandSolder; symbol Device:R_Small -> Pissbot-rescue:R_Small-Device
- R5, R6, R7: footprint (none) -> Resistor_SMD:R_0603_1608Metric_Pad1.05x0.95mm_HandSolder; symbol Device:R_Small -> Pissbot-rescue:R_Small-Device
- R8: renamed from R9; footprint (none) -> Resistor_SMD:R_0603_1608Metric_Pad1.05x0.95mm_HandSolder; symbol Device:R_Small -> Pissbot-rescue:R_Small-Device
- U1: footprint QFN28_5X5_SIL -> footprints:CP2102-GM
- U2: renamed from U3; footprint SOIC_DBVR_TEX -> TLV74033PDBVR:TLV74033PDBVR
- U3: renamed from U2; footprint DRL0006A -> TPS563231DRLR:TPS563231DRLR
Connections:
- net labels added: ELEMEMENT_1, ELEMENT1, ELEMENT2, ELEMENT_2, FAN, LED, PRODUCT_FLOW, REFLUX_FLOW, REFLUX_PUMP, RXD0, TXD0, UART1_RX, UART1_TX
- net labels removed: ESP_D+, ESP_D-, Element_1, Element_2, Fan, I2C-INT, I2C_INTA, I2C_INTB, I2C_SCL, I2C_SDA, LED1, PI_D+, PI_D-, Product_flow, Reflux_flow, SCL, SDA
- wire segments 257 -> 327
- no-connect marks 12 -> 38
Other:
- note added: "1Wire Temperature Sensor Bus"
- note added: "Boot/Reset Switches"
- note added: "Element Connectors"
- note added: "Fan Connector"
- note added: "Flowmeter Connectors"
- note added: "JTAG Header"
- note added: "Micro USB"
- note added: "Power Connector (12V)"
- note added: "Power Connectors"
- note added: "Power Supplies"
- note added: "Pump 1"
- note added: "Pump 2"
- note added: "Pump Drivers"
- note added: "Reverse Current Protection"
- note added: "Test Pads"
- note added: "USB to UART Bridge"
- note removed: "I2C Port Expander"
- note removed: "Ideal diode section for reverse current protection"
- note removed: "Micro USB connectors"
- note removed: "NOTE: Add reverse current diodes for power supplies"
- note removed: "Select I2C address 0x20"
- note removed: "TODO: Add RGB led on port B for indication?"
- moved on the sheet: J1, J10, J2, J3, J4, J5, J6, J7, J8
