File: Distiller Controller V6/Pissbot/Pissbot.sch (KiCad schematic (older format))
At the start: 34 parts, among them J1 Raspberry_Pi_2_3, U1 CP2102-GM, U2 TPS563231DRLR, U3 TLV74033PDBVR

Commit message: Updated PCB
Parts:
- removed C10, C9: 22uF, symbol Pissbot-rescue:C-Device
- removed C11: 0.1uF, symbol Pissbot-rescue:C-Device
- removed C3, C4, C5: 10uF, symbol Pissbot-rescue:C-Device
- removed C6, C8: 1uF, symbol Pissbot-rescue:C-Device
- removed D1: LED, symbol Pissbot-rescue:LED-Device
- removed R5: 73.2k, symbol Pissbot-rescue:R-Device
- removed R6: 10k, symbol Pissbot-rescue:R-Device
- removed R7: 1k, symbol Pissbot-rescue:R-Device
- removed R? (x2): 4.7k, symbol Pissbot-rescue:R-Device
- added A1: ESP32-WROVER-I, XCVR_ESP32-WROVER-I, symbol ESP32-WROVER-I:ESP32-WROVER-I
- added C10, C9, C?: 22uF, symbol Device:C_Small
- added C11, C? (x3): 0.1uF, symbol Device:C_Small
- added C3, C5, C6: 10uF, symbol Device:C_Small
- added C4, C8: 1uF, symbol Device:C_Small
- added D1: LED_Small, symbol Device:LED_Small
- added D? (x2): MBRD835TR, symbol Device:D_Schottky
- added D? (x3): 9.1V, symbol Device:D_Zener_Small_ALT
- added J?: MicroUSB_ESP, symbol Connector:USB_B_Micro
- added J?: MicroUSB_PI, symbol Connector:USB_B_Micro
- added Q? (x2): MCU80N03A-TP, symbol Device:Q_NMOS_GDS
- added Q? (x2): S8050, Package_TO_SOT_THT:TO-92_Inline, symbol Transistor_BJT:S8050
- added Q? (x3): SSM3J338R, SOT-23F_TOS, symbol SSM3J338R:SSM3J338R
- added R5: 73.2k, symbol Device:R_Small
- added R6, R? (x3): 10k, symbol Device:R_Small
- added R7, R8: 2k, symbol Device:R_Small
- added R9: 1k, symbol Device:R_Small
- added R? (x2): 4.7k, symbol Device:R_Small
- added R? (x3): 100k, symbol Device:R_Small
- added U?: MCP23017_ML, Package_DFN_QFN:QFN-28-1EP_6x6mm_P0.65mm_EP4.25x4.25mm, symbol Interface_Expansion:MCP23017_ML
- J2, J3, J4, J5, J6, J7, J8, J9: renamed from J?; symbol SM03B-SRSS-TB_LF__SN_:SM03B-SRSS-TB(LF)(SN) -> Pissbot-rescue:SM03B-SRSS-TB(LF)(SN)-SM03B-SRSS-TB_LF__SN_
- U1: symbol 2020-09-23_10-39-16:CP2102-GM -> Pissbot-rescue:CP2102-GM-2020-09-23_10-39-16
- U2: symbol 2020-09-23_08-56-15:TPS563231DRLR -> Pissbot-rescue:TPS563231DRLR-2020-09-23_08-56-15
- U3: symbol 2020-09-23_09-25-31:TLV74033PDBVR -> Pissbot-rescue:TLV74033PDBVR-2020-09-23_09-25-31
Connections:
- net labels added: 12V, 5V_IN, EN, ESP_D+, ESP_D-, ESP_VBUS, Element_1, Element_2, Fan, I2C-INT, I2C_INTA, I2C_INTB, I2C_SCL, I2C_SDA, IO0, IO2, IO4, IO5, JTAG-MTCK, JTAG-MTDI, JTAG-MTDO, JTAG-MTMS, LED1, P1_LOAD, P2_LOAD, PI_D+, PI_D-, PI_VBUS, PROD-PUMP, PROD_PUMP, Product_flow, REFLUX-PUMP, Reflux_flow, SCL, SDA, USB_D+, USB_D-
- net labels removed: USB_DN, USB_DP
- wire segments 143 -> 257
- no-connect marks 0 -> 12
Other:
- note added: "Boot magic. See ESP-32 Devkit C schematic"
- note added: "I2C Port Expander"
- note added: "Ideal diode section for reverse current protection"
- note added: "Micro USB connectors"
- note added: "NOTE: Add ESD protection"
- note added: "NOTE: Add reverse current protection for 5V power supplies"
- note added: "NOTE: Use P channel mosfet for reverse voltage protection"
- note added: "NOTE: Use zener to clamp gate-source voltage for 12v in?"
- note added: "Note: Is this the best way to drive the pumps?"
- note added: "Select I2C address 0x20"
- moved on the sheet: C7, L1, U2, U3

Commit message: Updated PCB. Added library files
Parts:
- removed C?: 0.1uF, symbol Device:C_Small
- removed J?: MicroUSB_PI, symbol Connector:USB_B_Micro
- removed R8: 2k, symbol Device:R_Small
- removed U?: MCP23017_ML, Package_DFN_QFN:QFN-28-1EP_6x6mm_P0.65mm_EP4.25x4.25mm, symbol Interface_Expansion:MCP23017_ML
- added J11, J12, J13: T4, JST-SH 3 Connector:JST_SM03B-SRSS-TB(LF)(SN), symbol Pissbot-rescue:SM03B-SRSS-TB(LF)(SN)-SM03B-SRSS-TB_LF__SN_
- added J14, J15: SM02B-SRSS-TB(LF)(SN), JST SH 2Pin:SM02B-SRSS-TB(LF)(SN), symbol SM02B-SRSS-TB_LF__SN_:SM02B-SRSS-TB(LF)(SN)
- added J16: Conn_01x02_Female, Connector_AMASS:AMASS_XT30PW-F_1x02_P2.50mm_Horizontal, symbol Connector:Conn_01x02_Female
- added J17, J18: Conn_01x02_Female, Screw Terminal - TB001:CUI_TB001-500-02BE, symbol Connector:Conn_01x02_Female
- added R17, R18, R19, R20, R?: 2k, Resistor_SMD:R_0603_1608Metric_Pad1.05x0.95mm_HandSolder, symbol Pissbot-rescue:R_Small-Device
- added U? (x2): PTS647SM38SMTR2LFS, SW_PTS647SM38SMTR2LFS_CNK, symbol TactileSwitch:PTS647SM38SMTR2LFS
- A1: footprint XCVR_ESP32-WROVER-I -> ESP32-WROVER-I:XCVR_ESP32-WROVER-I; symbol ESP32-WROVER-I:ESP32-WROVER-I -> Pissbot-rescue:ESP32-WROVER-I-ESP32-WROVER-I
- C1: footprint (none) -> Capacitor_SMD:C_0603_1608Metric
- C10, C11, C5, C6, C9: footprint (none) -> Capacitor_SMD:C_0603_1608Metric; symbol Device:C_Small -> Pissbot-rescue:C_Small-Device
- C12, C13, C14: renamed from C?; footprint (none) -> Capacitor_SMD:C_0603_1608Metric; symbol Device:C_Small -> Pissbot-rescue:C_Small-Device
- C2: renamed from C3; footprint (none) -> Capacitor_SMD:C_0603_1608Metric; symbol Device:C_Small -> Pissbot-rescue:C_Small-Device
- C3: renamed from C4; footprint (none) -> Capacitor_SMD:C_0603_1608Metric; symbol Device:C_Small -> Pissbot-rescue:C_Small-Device
- C4: renamed from C2; footprint (none) -> Capacitor_SMD:C_0603_1608Metric
- C7: renamed from C8; footprint (none) -> Capacitor_SMD:C_0603_1608Metric; symbol Device:C_Small -> Pissbot-rescue:C_Small-Device
- C8: renamed from C7; footprint (none) -> Capacitor_SMD:C_0603_1608Metric
- D1: footprint (none) -> LED_SMD:LED_0201_0603Metric; symbol Device:LED_Small -> Pissbot-rescue:LED_Small-Device
- D2, D3: renamed from D?; footprint (none) -> Package_TO_SOT_SMD:TO-252-2; symbol Device:D_Schottky -> Pissbot-rescue:D_Schottky-Device
- D4, D5, D6: renamed from D?; footprint (none) -> Package_TO_SOT_SMD:SOT-23; symbol Device:D_Zener_Small_ALT -> Pissbot-rescue:D_Zener_Small_ALT-Device
- J1: renamed from J2; footprint JST_SM03B-SRSS-TB(LF)(SN) -> JST-SH 3 Connector:JST_SM03B-SRSS-TB(LF)(SN)
- J10: renamed from J1; footprint (none) -> PiZero:ADA3708_RPI-ZERO
- J2: renamed from J3; footprint JST_SM03B-SRSS-TB(LF)(SN) -> JST-SH 3 Connector:JST_SM03B-SRSS-TB(LF)(SN)
- J3: renamed from J4; footprint JST_SM03B-SRSS-TB(LF)(SN) -> JST-SH 3 Connector:JST_SM03B-SRSS-TB(LF)(SN)
- J4: renamed from J5; footprint JST_SM03B-SRSS-TB(LF)(SN) -> JST-SH 3 Connector:JST_SM03B-SRSS-TB(LF)(SN)
- J5: renamed from J6; footprint JST_SM03B-SRSS-TB(LF)(SN) -> JST-SH 3 Connector:JST_SM03B-SRSS-TB(LF)(SN)
- J6: renamed from J7; footprint JST_SM03B-SRSS-TB(LF)(SN) -> JST-SH 3 Connector:JST_SM03B-SRSS-TB(LF)(SN)
- J7: renamed from J8; footprint JST_SM03B-SRSS-TB(LF)(SN) -> JST-SH 3 Connector:JST_SM03B-SRSS-TB(LF)(SN)
- J8: renamed from J9; footprint JST_SM03B-SRSS-TB(LF)(SN) -> JST-SH 3 Connector:JST_SM03B-SRSS-TB(LF)(SN)
- J9: renamed from J?; footprint (none) -> Micro USB:Micro-USB-TE_2040002-1; symbol Connector:USB_B_Micro -> Pissbot-rescue:USB_B_Micro-Connector
- L1: footprint (none) -> 3_3uH_ECSMPIL06303R3MC:ECS-MPIL0630-3R3MC
- Q1, Q2: renamed from Q?; footprint (none) -> Package_TO_SOT_SMD:TO-252-2; symbol Device:Q_NMOS_GDS -> Pissbot-rescue:Q_NMOS_GDS-Device
- Q3, Q4, Q5: renamed from Q?; footprint SOT-23F_TOS -> Package_TO_SOT_SMD:SOT-23; symbol SSM3J338R:SSM3J338R -> Pissbot-rescue:SSM3J338R-SSM3J338R
- Q6, Q7: renamed from Q?; footprint Package_TO_SOT_THT:TO-92_Inline -> Package_TO_SOT_SMD:SOT-23; symbol Transistor_BJT:S8050 -> Pissbot-rescue:S8050-Transistor_BJT
- R1, R2, R3, R4: footprint (none) -> Resistor_SMD:R_0603_1608Metric_Pad1.05x0.95mm_HandSolder
- R10, R11, R12, R13, R14, R15, R16, R9: renamed from R?; footprint (none) -> Resistor_SMD:R_0603_1608Metric_Pad1.05x0.95mm_HandSolder; symbol Device:R_Small -> Pissbot-rescue:R_Small-Device
- R5, R6, R7: footprint (none) -> Resistor_SMD:R_0603_1608Metric_Pad1.05x0.95mm_HandSolder; symbol Device:R_Small -> Pissbot-rescue:R_Small-Device
- R8: renamed from R9; footprint (none) -> Resistor_SMD:R_0603_1608Metric_Pad1.05x0.95mm_HandSolder; symbol Device:R_Small -> Pissbot-rescue:R_Small-Device
- U1: footprint QFN28_5X5_SIL -> footprints:CP2102-GM
- U2: renamed from U3; footprint SOIC_DBVR_TEX -> TLV74033PDBVR:TLV74033PDBVR
- U3: renamed from U2; footprint DRL0006A -> TPS563231DRLR:TPS563231DRLR
Connections:
- net labels added: ELEMEMENT_1, ELEMENT1, ELEMENT2, ELEMENT_2, FAN, LED, PRODUCT_FLOW, REFLUX_FLOW, REFLUX_PUMP, RXD0, TXD0, UART1_RX, UART1_TX
- net labels removed: ESP_D+, ESP_D-, Element_1, Element_2, Fan, I2C-INT, I2C_INTA, I2C_INTB, I2C_SCL, I2C_SDA, LED1, PI_D+, PI_D-, Product_flow, Reflux_flow, SCL, SDA
- wire segments 257 -> 327
- no-connect marks 12 -> 38
Other:
- note added: "1Wire Temperature Sensor Bus"
- note added: "Boot/Reset Switches"
- note added: "Fan Connector"
- note added: "Flowmeter Connectors"
- note added: "Micro USB"
- note added: "Power Connector (12V)"
- note added: "Power Supplies"
- note added: "Pump 1"
- note added: "Pump 2"
- note added: "Pump Drivers"
- note added: "Reverse Current Protection"
- note added: "Test Pads"
- note added: "USB to UART Bridge"
- note removed: "I2C Port Expander"
- note removed: "Ideal diode section for reverse current protection"
- note removed: "Micro USB connectors"
- note removed: "NOTE: Add reverse current diodes for power supplies"
- note removed: "Select I2C address 0x20"
- moved on the sheet: J1, J10, J2, J3, J4, J5, J6, J7, J8

Commit message: Save
Other:
- note added: "Element Connectors"
- note added: "JTAG Header"
- note added: "Power Connectors"
- moved on the sheet: J16, J17, J18
Changed lines of the file:
@@
 L Connector:Conn_01x02_Female J16
 U 1 1 606D1547
-P 12300 7150
-F 0 "J16" H 12328 7126 50  0000 L CNN
-F 1 "Conn_01x02_Female" H 12328 7035 50  0000 L CNN
-F 2 "Connector_AMASS:AMASS_XT30PW-F_1x02_P2.50mm_Horizontal" H 12300 7150 50  0001 C CNN
-F 3 "~" H 12300 7150 50  0001 C CNN
-	1    12300 7150
+P 12600 7000
+F 0 "J16" H 12628 6976 50  0000 L CNN
+F 1 "Conn_01x02_Female" H 12628 6885 50  0000 L CNN
+F 2 "Connector_AMASS:AMASS_XT30PW-F_1x02_P2.50mm_Horizontal" H 12600 7000 50  0001 C CNN
+F 3 "~" H 12600 7000 50  0001 C CNN
+	1    12600 7000
 	1    0    0    -1
 $EndComp
@@
 L Connector:Conn_01x02_Female J17
 U 1 1 606D19C7
-P 12300 7750
-F 0 "J17" H 12328 7726 50  0000 L CNN
-F 1 "Conn_01x02_Female" H 12328 7635 50  0000 L CNN
-F 2 "Screw Terminal - TB001:CUI_TB001-500-02BE" H 12300 7750 50  0001 C CNN
-F 3 "~" H 12300 7750 50  0001 C CNN
-	1    12300 7750
+P 12600 7600
+F 0 "J17" H 12628 7576 50  0000 L CNN
+F 1 "Conn_01x02_Female" H 12628 7485 50  0000 L CNN
+F 2 "Screw Terminal - TB001:CUI_TB001-500-02BE" H 12600 7600 50  0001 C CNN
+F 3 "~" H 12600 7600 50  0001 C CNN
+	1    12600 7600
 	1    0    0    -1
 $EndComp
@@
 L Connector:Conn_01x02_Female J18
 U 1 1 606D1EDD
-P 12300 8200
-F 0 "J18" H 12328 8176 50  0000 L CNN
-F 1 "Conn_01x02_Female" H 12328 8085 50  0000 L CNN
-F 2 "Screw Terminal - TB001:CUI_TB001-500-02BE" H 12300 8200 50  0001 C CNN
-F 3 "~" H 12300 8200 50  0001 C CNN
-	1    12300 8200
-	1    0    0    -1
-$EndComp
-Wire Wire Line
-	12100 7150 11800 7150
-Wire Wire Line
-	12100 7250 11800 7250
+P 12600 8050
+F 0 "J18" H 12628 8026 50  0000 L CNN
+F 1 "Conn_01x02_Female" H 12628 7935 50  0000 L CNN
+F 2 "Screw Terminal - TB001:CUI_TB001-500-02BE" H 12600 8050 50  0001 C CNN
+F 3 "~" H 12600 8050 50  0001 C CNN
+	1    12600 8050
+	1    0    0    -1
+$EndComp
+Wire Wire Line
+	12400 7000 12100 7000
+Wire Wire Line
+	12400 7100 12100 7100
 $Comp
 L Pissbot-rescue:+12V-power #PWR0109
 U 1 1 606FD685
-P 11800 7150
-F 0 "#PWR0109" H 11800 7000 50  0001 C CNN
-F 1 "+12V" V 11815 7278 50  0000 L CNN
-F 2 "" H 11800 7150 50  0001 C CNN
-F 3 "" H 11800 7150 50  0001 C CNN
-	1    11800 7150
+P 12100 7000
+F 0 "#PWR0109" H 12100 6850 50  0001 C CNN
+F 1 "+12V" V 12115 7128 50  0000 L CNN
+F 2 "" H 12100 7000 50  0001 C CNN
+F 3 "" H 12100 7000 50  0001 C CNN
+	1    12100 7000
 	0    -1   -1   0
 $EndComp
@@
 L Pissbot-rescue:GND-power #PWR0110
 U 1 1 606FE0A8
-P 11800 7250
-F 0 "#PWR0110" H 11800 7000 50  0001 C CNN
-F 1 "GND-power" H 12050 7150 50  0000 C CNN
-F 2 "" H 11800 7250 50  0001 C CNN
-F 3 "" H 11800 7250 50  0001 C CNN
-	1    11800 7250
-	1    0    0    -1
-$EndComp
-Text Notes 13050 7050 2    50   ~ 0
+P 12100 7100
+F 0 "#PWR0110" H 12100 6850 50  0001 C CNN
+F 1 "GND-power" H 12350 7000 50  0000 C CNN
+F 2 "" H 12100 7100 50  0001 C CNN
+F 3 "" H 12100 7100 50  0001 C CNN
+	1    12100 7100
+	1    0    0    -1
+$EndComp
+Text Notes 13350 6900 2    50   ~ 0
 Power Connector (12V)
 Wire Wire Line
-	12100 7750 11850 7750
-Wire Wire Line
-	12100 7850 11750 7850
+	12400 7600 12150 7600
+Wire Wire Line
+	12400 7700 12050 7700
 $Comp
 L Pissbot-rescue:+12V-power #PWR0111
 U 1 1 60740718
-P 11850 7750
-F 0 "#PWR0111" H 11850 7600 50  0001 C CNN
-F 1 "+12V" V 11865 7878 50  0000 L CNN
-F 2 "" H 11850 7750 50  0001 C CNN
-F 3 "" H 11850 7750 50  0001 C CNN
-	1    11850 7750
+P 12150 7600
+F 0 "#PWR0111" H 12150 7450 50  0001 C CNN
+F 1 "+12V" V 12165 7728 50  0000 L CNN
+F 2 "" H 12150 7600 50  0001 C CNN
+F 3 "" H 12150 7600 50  0001 C CNN
+	1    12150 7600
 	0    -1   -1   0
 $EndComp
-Text Label 11750 7850 0    50   ~ 0
+Text Label 12050 7700 0    50   ~ 0
 P1_LOAD
 Wire Wire Line
-	12100 8200 11750 8200
-Wire Wire Line
-	12100 8300 11750 8300
+	12400 8050 12050 8050
+Wire Wire Line
+	12400 8150 12050 8150
 $Comp
 L Pissbot-rescue:+12V-power #PWR0112
 U 1 1 607AFA27
-P 11750 8200
-F 0 "#PWR0112" H 11750 8050 50  0001 C CNN
-F 1 "+12V" V 11765 8328 50  0000 L CNN
-F 2 "" H 11750 8200 50  0001 C CNN
-F 3 "" H 11750 8200 50  0001 C CNN
-	1    11750 8200
+P 12050 8050
+F 0 "#PWR0112" H 12050 7900 50  0001 C CNN
+F 1 "+12V" V 12065 8178 50  0000 L CNN
+F 2 "" H 12050 8050 50  0001 C CNN
+F 3 "" H 12050 8050 50  0001 C CNN
+	1    12050 8050
 	0    -1   -1   0
 $EndComp
-Text Label 11750 8300 0    50   ~ 0
+Text Label 12050 8150 0    50   ~ 0
 P2_LOAD
-Text Notes 12150 7650 0    50   ~ 0
+Text Notes 12450 7500 0    50   ~ 0
 Pump 1
-Text Notes 12150 8100 0    50   ~ 0
+Text Notes 12450 7950 0    50   ~ 0
 Pump 2
 Wire Wire Line
@@
 Text Notes 9050 8600 0    50   ~ 0
 Test Pads
+Wire Notes Line
+	8950 9600 11800 9600
+Text Notes 9050 9800 0    50   ~ 0
+JTAG Header
+Text Notes 9050 6750 0    50   ~ 0
+Element Connectors
+Text Notes 11050 6750 0    50   ~ 0
+Power Connectors
 $EndSCHEMATC
